File: LED-Matrix/Eagle/LEDMatrixi.sch (EAGLE design)
At the start: 70 parts, among them IC1 MAX7219CWG

Commit message: Sletta fasit
Detaljar i "Notes"
Parts:
- removed DATAOUT: 2x5, Wurth_Elektronik_Electromechanic_Board_to_Board_Connectors_rev16a:610X1021121
- removed LED10, LED11, LED12, LED13, LED14, LED15, LED16, LED17, LED18, LED19, LED2, LED20, LED21, LED22, LED23, LED24, LED25, LED26, LED27, LED28, LED29, LED3, LED30, LED31, LED32, LED33, LED34, LED35, LED36, LED37, LED38, LED39, LED4, LED40, LED41, LED42, LED43, LED44, LED45, LED46, LED47, LED48, LED49, LED5, LED50, LED51, LED52, LED53, LED54, LED55, LED56, LED57, LED58, LED59, LED6, LED60, LED61, LED62, LED63, LED64, LED7, LED8, LED9: SMT 1206, led:LEDCHIPLED_1206
Connections:
- removed net CLK: DATAIN.7, DATAOUT.7, IC1.CLK
- removed net DIG0: IC1.DIG0, LED1.C, LED17.C, LED25.C, LED33.C, LED41.C, LED49.C, LED57.C, LED9.C
- removed net DIG1: IC1.DIG1, LED10.C, LED18.C, LED2.C, LED26.C, LED34.C, LED42.C, LED50.C, LED58.C
- removed net DIG2: IC1.DIG2, LED11.C, LED19.C, LED27.C, LED3.C, LED35.C, LED43.C, LED51.C, LED59.C
- removed net DIG3: IC1.DIG3, LED12.C, LED20.C, LED28.C, LED36.C, LED4.C, LED44.C, LED52.C, LED60.C
- removed net DIG4: IC1.DIG4, LED13.C, LED21.C, LED29.C, LED37.C, LED45.C, LED5.C, LED53.C, LED61.C
- removed net DIG5: IC1.DIG5, LED14.C, LED22.C, LED30.C, LED38.C, LED46.C, LED54.C, LED6.C, LED62.C
- removed net DIG6: IC1.DIG6, LED15.C, LED23.C, LED31.C, LED39.C, LED47.C, LED55.C, LED63.C, LED7.C
- removed net DIG7: IC1.DIG7, LED16.C, LED24.C, LED32.C, LED40.C, LED48.C, LED56.C, LED64.C, LED8.C
- removed net DIN: DATAIN.5, IC1.DIN
- removed net DOUT: DATAOUT.5, IC1.DOUT
- removed net GND: C1.-, C2.2, DATAIN.10, DATAIN.8, DATAIN.9, DATAOUT.10, DATAOUT.8, DATAOUT.9, IC1.GND_1, IC1.GND_2
- removed net LOAD: DATAIN.4, DATAOUT.4, IC1.LOAD
- removed net N$2: IC1.ISET, R1.1
- removed net SEGA: IC1.SEGA, LED10.A, LED11.A, LED12.A, LED13.A, LED14.A, LED15.A, LED16.A, LED9.A
- removed net SEGB: IC1.SEGB, LED17.A, LED18.A, LED19.A, LED20.A, LED21.A, LED22.A, LED23.A, LED24.A
- removed net SEGC: IC1.SEGC, LED25.A, LED26.A, LED27.A, LED28.A, LED29.A, LED30.A, LED31.A, LED32.A
- removed net SEGD: IC1.SEGD, LED33.A, LED34.A, LED35.A, LED36.A, LED37.A, LED38.A, LED39.A, LED40.A
- removed net SEGDP: IC1.SEGDP, LED1.A, LED2.A, LED3.A, LED4.A, LED5.A, LED6.A, LED7.A, LED8.A
- removed net SEGE: IC1.SEGE, LED41.A, LED42.A, LED43.A, LED44.A, LED45.A, LED46.A, LED47.A, LED48.A
- removed net SEGF: IC1.SEGF, LED49.A, LED50.A, LED51.A, LED52.A, LED53.A, LED54.A, LED55.A, LED56.A
- removed net SEGG: IC1.SEGG, LED57.A, LED58.A, LED59.A, LED60.A, LED61.A, LED62.A, LED63.A, LED64.A
- removed net VCC: C1.+, C2.1, DATAIN.1, DATAIN.2, DATAIN.3, DATAOUT.1, DATAOUT.2, DATAOUT.3, IC1.V+, R1.2
Other:
- note removed: "https://grabcad.com/library/capacitor-collection-electrolytic-vertical-mount-1/details?folder_id=5644801"
- moved on the sheet: DATAIN, LED1, R1
